Commit message: [UPD] update collision with primitive shapes

File: realsense2_description/urdf/_d405.urdf.xacro (robot description, xacro)
@@ -64,5 +64,6 @@
       </visual>
       <collision>
-        <origin xyz="0 ${-d405_cam_depth_py} 0" rpy="0 0 0"/>
+        <origin xyz="${d405_zero_depth_to_glass + d405_glass_to_front - d405_cam_depth/2} ${-d405_cam_depth_py} 0" rpy="0 0 0"/>
+        <!-- <origin xyz="0 ${-d405_cam_depth_py} 0" rpy="0 0 0"/> -->
         <geometry>
           <box size="${d405_cam_depth} ${d405_cam_width} ${d405_cam_height}"/>

Commit message: [FIX] add proper inertia

File: realsense2_description/urdf/_d405.urdf.xacro (robot description, xacro)
@@ -10,5 +10,5 @@
   <xacro:include filename="$(find realsense2_description)/urdf/_materials.urdf.xacro" />
   <xacro:macro name="sensor_d405" params="parent *origin name:=camera use_nominal_extrinsics:=false use_mesh:=true">
-    <xacro:property name="M_PI" value="3.1415926535897931" />
+    <xacro:property name="M_PI" value="3.14159" />
     <!-- The following values are approximate, and the camera node
      publishing TF values with actual calibrated camera extrinsic values -->
@@ -73,6 +73,8 @@
         <!-- The following are not reliable values, and should not be used for modeling -->
         <mass value="0.072" />
-        <origin xyz="0 0 0" />
-        <inertia ixx="0.003881243" ixy="0.0" ixz="0.0" iyy="0.000498940" iyz="0.0" izz="0.003879257" />
+        <origin xyz="${d405_zero_depth_to_glass + d405_glass_to_front - d405_cam_depth/2} ${-d405_cam_depth_py} 0" rpy="0 0 0"/>
+        <inertia ixx="${1/12*0.072*(d405_cam_depth**2+d405_cam_height**2)}" ixy="0.0" ixz="0.0"
+                 iyy="${1/12*0.072*(d405_cam_width**2+d405_cam_height**2)}" iyz="0.0"
+                 izz="${1/12*0.072*(d405_cam_depth**2+d405_cam_width**2)}" />
       </inertial>
     </link>

Commit message: [FIX] change d405 mass

File: realsense2_description/urdf/_d405.urdf.xacro (robot description, xacro)
@@ -72,9 +72,9 @@
       <inertial>
         <!-- The following are not reliable values, and should not be used for modeling -->
-        <mass value="0.072" />
+        <mass value="0.06" />
         <origin xyz="${d405_zero_depth_to_glass + d405_glass_to_front - d405_cam_depth/2} ${-d405_cam_depth_py} 0" rpy="0 0 0"/>
-        <inertia ixx="${1/12*0.072*(d405_cam_depth**2+d405_cam_height**2)}" ixy="0.0" ixz="0.0"
-                 iyy="${1/12*0.072*(d405_cam_width**2+d405_cam_height**2)}" iyz="0.0"
-                 izz="${1/12*0.072*(d405_cam_depth**2+d405_cam_width**2)}" />
+        <inertia ixx="${1/12*0.06*(d405_cam_depth**2+d405_cam_height**2)}" ixy="0.0" ixz="0.0"
+                 iyy="${1/12*0.06*(d405_cam_width**2+d405_cam_height**2)}" iyz="0.0"
+                 izz="${1/12*0.06*(d405_cam_depth**2+d405_cam_width**2)}" />
       </inertial>
     </link>

Commit message: [FIX] use find command to locate mesh file when using gz sim

File: realsense2_description/urdf/_d405.urdf.xacro (robot description, xacro)
@@ -66,5 +66,5 @@
         <origin xyz="${d405_zero_depth_to_glass + d405_glass_to_front} ${-d405_cam_depth_py} 0" rpy="${M_PI/2} 0 ${M_PI/2}"/>
         <geometry>
-	        <mesh filename="package://realsense2_description/meshes/d405.stl" scale="0.001 0.001 0.001" />
+	        <mesh filename="file://$(find realsense2_description)/meshes/d405.stl" scale="0.001 0.001 0.001" />
         </geometry>
         <material name="aluminum"/>

File: realsense2_description/urdf/_d415.urdf.xacro (robot description, xacro)
@@ -59,5 +59,5 @@
           <origin xyz="${d415_cam_mount_from_center_offset} ${-d415_cam_depth_py} 0" rpy="${M_PI/2} 0 ${M_PI/2}"/>
           <geometry>
-            <mesh filename="package://realsense2_description/meshes/d415.stl" />
+            <mesh filename="file://$(find realsense2_description)/meshes/d415.stl" />
           </geometry>
           <material name="aluminum"/>

File: realsense2_description/urdf/_d435.urdf.xacro (robot description, xacro)
@@ -66,5 +66,5 @@
           <origin xyz="${d435_zero_depth_to_glass + d435_glass_to_front} ${-d435_cam_depth_py} 0" rpy="${M_PI/2} 0 ${M_PI/2}"/>
           <geometry>
-            <mesh filename="package://realsense2_description/meshes/d435.dae" />
+            <mesh filename="file://$(find realsense2_description)/meshes/d435.dae" />
           </geometry>
         </xacro:if>

File: realsense2_description/urdf/_d436.urdf.xacro (robot description, xacro)
@@ -66,5 +66,5 @@
           <origin xyz="${d436_zero_depth_to_glass + d436_glass_to_front} ${-d436_cam_depth_py} 0" rpy="${M_PI/2} 0 ${M_PI/2}"/>
           <geometry>
-            <mesh filename="package://realsense2_description/meshes/d435.dae" />
+            <mesh filename="file://$(find realsense2_description)/meshes/d435.dae" />
           </geometry>
         </xacro:if>

File: realsense2_description/urdf/_d455.urdf.xacro (robot description, xacro)
@@ -68,5 +68,5 @@
         <geometry>
           <!-- <box size="${d455_cam_depth} ${d455_cam_width} ${d455_cam_height}"/> -->
-	        <mesh filename="package://realsense2_description/meshes/d455.stl" scale="0.001 0.001 0.001" />
+	        <mesh filename="file://$(find realsense2_description)/meshes/d455.stl" scale="0.001 0.001 0.001" />
         </geometry>
         <material name="aluminum"/>

File: realsense2_description/urdf/_d585.urdf.xacro (robot description, xacro)
@@ -67,5 +67,5 @@
         <geometry>
           <!-- <box size="${d585_cam_depth} ${d585_cam_width} ${d585_cam_height}"/> -->
-	        <mesh filename="package://realsense2_description/meshes/d585.stl" scale="0.001 0.001 0.001" />
+	        <mesh filename="file://$(find realsense2_description)/meshes/d585.stl" scale="0.001 0.001 0.001" />
         </geometry>
         <material name="aluminum"/>

File: realsense2_description/urdf/_r410.urdf.xacro (robot description, xacro)
@@ -51,5 +51,5 @@
         <geometry>
           <box size="${r410_cam_width} ${r410_cam_height} ${r410_cam_depth}"/>
-          <!--<mesh filename="package://realsense2_description/meshes/r410/r410.dae" />-->
+          <!--<mesh filename="file://$(find realsense2_description)/meshes/r410/r410.dae" />-->
         </geometry>
         <material name="aluminum"/>

File: realsense2_description/urdf/_r430.urdf.xacro (robot description, xacro)
@@ -51,5 +51,5 @@
         <geometry>
           <box size="${r430_cam_width} ${r430_cam_height} ${r430_cam_depth}"/>
-          <!--<mesh filename="package://realsense2_description/meshes/r430/r430.dae" />-->
+          <!--<mesh filename="file://$(find realsense2_description)/meshes/r430/r430.dae" />-->
         </geometry>
         <material name="aluminum"/>

File: realsense2_description/urdf/_usb_plug.urdf.xacro (robot description, xacro)
@@ -33,5 +33,5 @@
         <geometry>
           <!--box size="0.044850 0.008 0.0185" /-->
-          <mesh filename="package://realsense2_description/meshes/plug.stl" />
+          <mesh filename="file://$(find realsense2_description)/meshes/plug.stl" />
         </geometry>
         <material name="plastic"/>
@@ -41,5 +41,5 @@
         <geometry>
           <!--box size="0.044850 0.008 0.0185" /-->
-          <mesh filename="package://realsense2_description/meshes/plug_collision.stl" />
+          <mesh filename="file://$(find realsense2_description)/meshes/plug_collision.stl" />
         </geometry>
       </collision>
